Commit message: Train and steer scripts

File: autocone_description/urdf/colin.urdf.xacro (robot description, xacro)
@@ -39,4 +39,5 @@
     <!-- Update rate -->
     <xacro:property name="update_rate" value="30.0"/>
+    <xacro:property name="bumper_update_rate" value="30.0"/>
     <!-- Degree-to-radian conversions -->
     <xacro:property name="degrees_45" value="0.785398163"/>
@@ -454,5 +455,5 @@
                 channels, which at that point lie in the range [0,1]. -->
             <mean>0.0</mean>
-            <stddev>0.007</stddev>
+            <!--<stddev>0.007</stddev>-->
             </noise>
         </camera>
@@ -509,5 +510,5 @@
         <sensor name="bumper_sensor" type="contact">
             <always_on>true</always_on>
-            <update_rate>${update_rate}</update_rate>
+            <update_rate>${bumper_update_rate}</update_rate>
             <contact>
                 <collision>base_link_fixed_joint_lump__bumper_link_collision</collision>

Commit message: From stash

File: autocone_description/urdf/colin.urdf.xacro (robot description, xacro)
@@ -37,7 +37,10 @@
         chassis_wheeltrack along the y axis (distance between left and right wheels)
     -->
-    <!-- Update rate -->
-    <xacro:property name="update_rate" value="30.0"/>
+    <!-- Bumpper sensor Properties -->
     <xacro:property name="bumper_update_rate" value="30.0"/>
+    <!-- Camera Properties -->
+    <xacro:property name="cam_update_rate" value="30.0"/>
+    <xacro:property name="clipping_near" value="0.02"/>
+    <xacro:property name="clipping_far" value="3.0"/>
     <!-- Degree-to-radian conversions -->
     <xacro:property name="degrees_45" value="0.785398163"/>
@@ -437,15 +440,15 @@
     <gazebo reference="camera_link">
         <sensor type="camera" name="camera1">
-        <update_rate>${update_rate}</update_rate>
+        <update_rate>${cam_update_rate}</update_rate>
         <camera name="head">
             <horizontal_fov>1,0472</horizontal_fov>
             <image>
-            <width>800</width>
-            <height>800</height>
+            <width>1280</width>
+            <height>960</height>
             <format>R8G8B8</format>
             </image>
             <clip>
-            <near>0.02</near>
-            <far>300</far>
+            <near>${clipping_near}</near>
+            <far>${clipping_far}</far>
             </clip>
             <noise>

Commit message: Arruamando train_control ...

File: autocone_description/urdf/colin.urdf.xacro (robot description, xacro)
@@ -38,5 +38,5 @@
     -->
     <!-- Bumpper sensor Properties -->
-    <xacro:property name="bumper_update_rate" value="30.0"/>
+    <xacro:property name="bumper_update_rate" value="10.0"/>
     <!-- Camera Properties -->
     <xacro:property name="cam_update_rate" value="30.0"/>

Commit message: Finish datalogger

File: autocone_description/urdf/colin.urdf.xacro (robot description, xacro)
@@ -38,5 +38,5 @@
     -->
     <!-- Bumpper sensor Properties -->
-    <xacro:property name="bumper_update_rate" value="10.0"/>
+    <xacro:property name="bumper_update_rate" value="30.0"/>
     <!-- Camera Properties -->
     <xacro:property name="cam_update_rate" value="30.0"/>
@@ -56,5 +56,5 @@
     <xacro:property name="hitbox_length" value="0.370"/>
     <xacro:property name="hitbox_width" value="0.25"/>
-    <xacro:property name="hitbox_height" value="0.02"/>
+    <xacro:property name="hitbox_height" value="0.01"/>
     <!-- battery_dist is the distance between the inner edges of the
         batteries. battery_comp_depth is the battery compartment depth.

Commit message: Fix vision problems + other little things - fix problems to encode binary image before save

File: autocone_description/urdf/colin.urdf.xacro (robot description, xacro)
@@ -42,5 +42,5 @@
     <xacro:property name="cam_update_rate" value="30.0"/>
     <xacro:property name="clipping_near" value="0.02"/>
-    <xacro:property name="clipping_far" value="3.0"/>
+    <xacro:property name="clipping_far" value="1.5"/>
     <!-- Degree-to-radian conversions -->
     <xacro:property name="degrees_45" value="0.785398163"/>

Commit message: load city to gazebo

File: autocone_description/urdf/colin.urdf.xacro (robot description, xacro)
@@ -42,5 +42,5 @@
     <xacro:property name="cam_update_rate" value="30.0"/>
     <xacro:property name="clipping_near" value="0.02"/>
-    <xacro:property name="clipping_far" value="1.5"/>
+    <xacro:property name="clipping_far" value="10.5"/>
     <!-- Degree-to-radian conversions -->
     <xacro:property name="degrees_45" value="0.785398163"/>
